File: GateLinkMaster.kicad_pcb (KiCad board)
At the start: 2 copper layers, 9 parts, among them P1 USB_C_Plug_USB2.0, U1 ESP32-WROOM-32, U2 LM2576HVS-3.3

Commit message: CP2102
Parts:
- added C2: 10uF, Capacitor_SMD:C_0805_2012Metric_Pad1.18x1.45mm_HandSolder, F.Cu at (133.6, 132.3)
- added C3: 0.1uF, Capacitor_SMD:C_0805_2012Metric_Pad1.18x1.45mm_HandSolder, F.Cu at (133.6, 135.4)
- added C4: 10uF, Capacitor_SMD:C_0805_2012Metric_Pad1.18x1.45mm_HandSolder, F.Cu at (133.6, 138.4)
- added C5: 0.1uF, Capacitor_SMD:C_0805_2012Metric_Pad1.18x1.45mm_HandSolder, F.Cu at (133.6, 141.4)
- added C6: 10uF, Capacitor_SMD:C_0201_0603Metric, F.Cu at (104.4, 128.5)
- added C7: 1uF/16V, Capacitor_SMD:C_0201_0603Metric, F.Cu at (107.1, 134.2)
- added Q1: SS8050, Package_TO_SOT_SMD:SOT-23, F.Cu at (114.1, 123.1)
- added Q2: SS8550, Package_TO_SOT_SMD:SOT-23, F.Cu at (118.6, 123.1)
- added R2: 10k, Resistor_SMD:R_0201_0603Metric_Pad0.64x0.40mm_HandSolder, F.Cu at (128.0, 132.6)
- added R3: 1k, Resistor_SMD:R_0201_0603Metric_Pad0.64x0.40mm_HandSolder, F.Cu at (128.0, 134.4)
- added R4: 47.5K, Resistor_SMD:R_0201_0603Metric_Pad0.64x0.40mm_HandSolder, F.Cu at (128.0, 136.1)
- added R5: 22.1K, Resistor_SMD:R_0201_0603Metric_Pad0.64x0.40mm_HandSolder, F.Cu at (128.0, 137.9)
- added R6: 10K, Resistor_SMD:R_0201_0603Metric_Pad0.64x0.40mm_HandSolder, F.Cu at (128.0, 139.6)
- added R7: 10K, Resistor_SMD:R_0201_0603Metric_Pad0.64x0.40mm_HandSolder, F.Cu at (128.0, 141.4)
- added U3: SGM2212-3.3XKC3G/TR, SGM2212-3.3XKC3G/TR:SOT-223-3_SGM2212_SNC, F.Cu at (105.5, 122.2)
- C1: value C -> 1uF; footprint Capacitor_SMD:CP_Elec_3x5.3 -> Capacitor_SMD:C_0805_2012Metric_Pad1.18x1.45mm_HandSolder
- D4: footprint Diode_THT:D_DO-41_SOD81_P10.16mm_Horizontal -> Diode_SMD:D_0201_0603Metric
- U2: value LM2576HVS-3.3 -> CP2102N-Axx-xQFN28; footprint Package_TO_SOT_SMD:TO-263-5_TabPin3 -> Package_DFN_QFN:QFN-28-1EP_5x5mm_P0.5mm_EP3.35x3.35mm
- moved C1 90.5 mm to (133.6, 129.3), turned to 0 degrees
- moved D4 67.8 mm to (109.8, 132.5)
- moved D1 62.0 mm to (107.8, 132.5), turned to 0 degrees
- moved U1 59.4 mm to (109.9, 106.8), turned to 90 degrees
- moved D3 59.3 mm to (108.5, 134.2), turned to 0 degrees
- moved D2 58.6 mm to (110.0, 134.2), turned to 0 degrees
- moved R1 58.3 mm to (105.2, 134.2), turned to 0 degrees
- moved P1 57.2 mm to (105.5, 140.8)
- moved U2 53.2 mm to (116.4, 139.2), turned to -90 degrees
Connections:
- C1 pad 1: +3V3 -> Net-(U1-EN)
- D1 pad 2: +5V -> /VBUS
- D4 pad 2: +5V -> /VBUS
- P1 pad A4: +5V -> /VBUS
- P1 pad A9: +5V -> /VBUS
- P1 pad B4: +5V -> /VBUS
- P1 pad B9: +5V -> /VBUS
- U1 pad 3: unconnected-(U1-EN-Pad3) -> Net-(U1-EN)
- U2 pad 1: +5V -> unconnected-(U2-~{DCD}-Pad1)
- U2 pad 2: +3V3 -> unconnected-(U2-~{RI}/CLK-Pad2)
- U2 pad 4: unconnected-(U2-FB-Pad4) -> /USB_DP
- U2 pad 5: unconnected-(U2-~{ON}/OFF-Pad5) -> /USB_DN
Routing:
- net GND: track 126.4 -> 4.13 mm
- net +3V3: track 50.6 -> 3.01 mm, vias 2 -> 0
- net +5V: track 36.0 -> 0.00 mm, vias 1 -> 0
- net Net-(Q2-B): track 0.00 -> 23.7 mm
- net Net-(P1-CC): track 7.09 -> 0.00 mm
Other:
- board outline added: 36.5 x 48.3 mm
