File: GateLinkMaster.kicad_sch (KiCad schematic)
At the start: 9 parts, among them P1 USB_C_Plug_USB2.0, U1 ESP32-WROOM-32, U2 LM2576HVS-3.3

Commit message: CP2102
Parts:
- removed U2: LM2576HVS-3.3, Package_TO_SOT_SMD:TO-263-5_TabPin3, symbol Regulator_Switching:LM2576HVS-3.3
- added C2, C4: 10uF, Capacitor_SMD:C_0805_2012Metric_Pad1.18x1.45mm_HandSolder, symbol Device:C
- added C3, C5: 0.1uF, Capacitor_SMD:C_0805_2012Metric_Pad1.18x1.45mm_HandSolder, symbol Device:C
- added C6: 10uF, Capacitor_SMD:C_0201_0603Metric, symbol Device:C
- added C7: 1uF/16V, Capacitor_SMD:C_0201_0603Metric, symbol Device:C
- added Q1: SS8050, Package_TO_SOT_SMD:SOT-23, symbol Transistor_BJT:SS8050
- added Q2: SS8550, Package_TO_SOT_SMD:SOT-23, symbol Transistor_BJT:SS8550
- added R2: 10k, Resistor_SMD:R_0201_0603Metric_Pad0.64x0.40mm_HandSolder, symbol Device:R
- added R3: 1k, Resistor_SMD:R_0201_0603Metric_Pad0.64x0.40mm_HandSolder, symbol Device:R
- added R4: 47.5K, Resistor_SMD:R_0201_0603Metric_Pad0.64x0.40mm_HandSolder, symbol Device:R
- added R5: 22.1K, Resistor_SMD:R_0201_0603Metric_Pad0.64x0.40mm_HandSolder, symbol Device:R
- added R6, R7: 10K, Resistor_SMD:R_0201_0603Metric_Pad0.64x0.40mm_HandSolder, symbol Device:R
- added U2: CP2102N-Axx-xQFN28, Package_DFN_QFN:QFN-28-1EP_5x5mm_P0.5mm_EP3.35x3.35mm, symbol Interface_USB:CP2102N-Axx-xQFN28
- added U3: SGM2212-3.3XKC3G/TR, SOT-223-3_SGM2212_SNC, symbol SGM2212-3.3XKC3G/TR:SGM2212-3.3XKC3G_TR
- C1: value C -> 1uF; footprint Capacitor_SMD:CP_Elec_3x5.3 -> Capacitor_SMD:C_0805_2012Metric_Pad1.18x1.45mm_HandSolder
- D4: footprint Diode_THT:D_DO-41_SOD81_P10.16mm_Horizontal -> Diode_SMD:D_0201_0603Metric
Connections:
- net +3V3: now also C4.1, C5.1, C6.1, R3.1, U2.6 (VDD), U2.7 (VREGIN), U3.2 (VOUT); no longer C1.1
- net +5V: now also C2.1, C3.1, U3.3 (VIN); no longer D1.2 (A2), D4.2 (A), P1.A4 (VBUS), P1.A9 (VBUS), P1.B4 (VBUS), P1.B9 (VBUS)
- net GND: now also C2.2, C3.2, C4.2, C5.2, C6.2, C7.2, R2.2, R4.2, U2.29 (GND), U2.3 (GND), U3.1 (GND)
- net USB_DN: now also U2.5 (D-)
- net USB_DP: now also U2.4 (D+)
- net at U1.3 (EN): now also C1.1
- new net: Q2.1 (B), R7.2
- new net: Q1.1 (B), R6.2
- new net: R2.1, U2.11 (~{SUSPEND})
- new net: C7.1, R4.1, R5.2, U2.8 (VBUS)
- new net: R3.2, U2.9 (~{RST})
- new net DTR: Q2.3 (C), R6.1, U2.28 (~{DTR})
- new net ESP_RST: Q1.3 (C)
- new net GPIO0: Q2.2 (E)
- new net RTS: Q1.2 (E), R7.1, U2.24 (~{RTS})
- new net U0RXD: U2.26 (TXD)
- new net U0TXD: U2.25 (RXD)
- new net VBUS: D1.2 (A2), D4.2 (A), P1.A4 (VBUS), P1.A9 (VBUS), P1.B4 (VBUS), P1.B9 (VBUS), R5.1
Other:
- note added: "5V-3.3V"
- note added: "USB-Port"
- moved on the sheet: D1, D2, D3, D4, P1, R1, U1

Commit message: jesus
Parts:
- removed D1, D2, D3: D_TVS, Diode_SMD:Nexperia_DSN0603-2_0.6x0.3mm_P0.4mm, symbol Device:D_TVS
- removed U3: SGM2212-3.3XKC3G/TR, SOT-223-3_SGM2212_SNC, symbol SGM2212-3.3XKC3G/TR:SGM2212-3.3XKC3G_TR
- added D1: 1N4148, Diode_THT:D_DO-35_SOD27_P7.62mm_Horizontal, symbol Diode:1N4148
- added D2: D_Schottky, Diode_SMD:D_SMA, symbol Device:D_Schottky
- added L1: 15uH, Inductor_SMD:L_6.3x6.3_H3, symbol Device:L
- added R8: 31.6k, Resistor_SMD:R_0603_1608Metric, symbol Device:R
- added R9: 10k, Resistor_SMD:R_0603_1608Metric, symbol Device:R
- added U4: USBLC6-2SC6, Package_TO_SOT_SMD:SOT-23-6, symbol Power_Protection:USBLC6-2SC6
- added U5: MCP16301x-xCH, Package_TO_SOT_SMD:SOT-23-6, symbol Regulator_Switching:MCP16301x-xCH
- C2: footprint Capacitor_SMD:C_0805_2012Metric_Pad1.18x1.45mm_HandSolder -> Capacitor_SMD:C_0805_2012Metric
- C3: value 0.1uF -> 100nF; footprint Capacitor_SMD:C_0805_2012Metric_Pad1.18x1.45mm_HandSolder -> Capacitor_SMD:C_0603_1608Metric
- C4: value 10uF -> 10u; footprint Capacitor_SMD:C_0805_2012Metric_Pad1.18x1.45mm_HandSolder -> Capacitor_SMD:C_0603_1608Metric
- C5: value 0.1uF -> 10u; footprint Capacitor_SMD:C_0805_2012Metric_Pad1.18x1.45mm_HandSolder -> Capacitor_SMD:C_0603_1608Metric
- R1: value 5.1k -> 5.1K; footprint Resistor_SMD:R_0201_0603Metric -> Resistor_SMD:R_0603_1608Metric
Connections:
- net +3V3: now also D1.2 (A), L1.2, R8.1
- net GND: now also D2.2 (A), R9.2, U4.2 (GND), U5.2 (GND); no longer C3.2
- net USB_DN: now also U4.6 (I/O1); no longer P1.A7 (D-)
- net USB_DP: now also U4.4 (I/O2); no longer P1.A6 (D+)
- net VBUS: now also C2.1, U4.5 (VBUS), U5.4 (EN), U5.5 (V_{IN})
- net +5V: no longer names the net of C3.1
- net +5V: now also D1.1 (K), U5.1 (BOOST); no longer C2.1
- new net: R8.2, R9.1, U5.3 (Vfb)
- new net: C3.2, D2.1 (K), L1.1, U5.6 (SW)
- new net: P1.A7 (D-), U4.1 (I/O1)
- new net: P1.A6 (D+), U4.3 (I/O2)
