File: GateLinkMaster.kicad_sch (KiCad schematic)
At the start: 27 parts, among them P1 USB_C_Plug_USB2.0, Q1 SS8050, Q2 SS8550, U1 ESP32-WROOM-32, U2 CP2102N-Axx-xQFN28, U4 USBLC6-2SC6, U5 MCP16301x-xCH

Commit message: Update to new project layout Begin new schematic
Parts:
- removed C1: 1uF, Capacitor_SMD:C_0805_2012Metric_Pad1.18x1.45mm_HandSolder, symbol Device:C
- removed C2: 10uF, Capacitor_SMD:C_0805_2012Metric, symbol Device:C
- removed C3: 100nF, Capacitor_SMD:C_0603_1608Metric, symbol Device:C
- removed C4, C5: 10u, Capacitor_SMD:C_0603_1608Metric, symbol Device:C
- removed C6: 10uF, Capacitor_SMD:C_0201_0603Metric, symbol Device:C
- removed C7: 1uF/16V, Capacitor_SMD:C_0201_0603Metric, symbol Device:C
- removed D1: 1N4148, Diode_THT:D_DO-35_SOD27_P7.62mm_Horizontal, symbol Diode:1N4148
- removed D2: D_Schottky, Diode_SMD:D_SMA, symbol Device:D_Schottky
- removed D4: 1N5819, Diode_SMD:D_0201_0603Metric, symbol Diode:1N5819
- removed L1: 15uH, Inductor_SMD:L_6.3x6.3_H3, symbol Device:L
- removed P1: USB_C_Plug_USB2.0, Connector_USB:USB_C_Receptacle_G-Switch_GT-USB-7010ASV, symbol Connector:USB_C_Plug_USB2.0
- removed Q1: SS8050, Package_TO_SOT_SMD:SOT-23, symbol Transistor_BJT:SS8050
- removed Q2: SS8550, Package_TO_SOT_SMD:SOT-23, symbol Transistor_BJT:SS8550
- removed R1: 5.1K, Resistor_SMD:R_0603_1608Metric, symbol Device:R
- removed R2: 10k, Resistor_SMD:R_0201_0603Metric_Pad0.64x0.40mm_HandSolder, symbol Device:R
- removed R3: 1k, Resistor_SMD:R_0201_0603Metric_Pad0.64x0.40mm_HandSolder, symbol Device:R
- removed R4: 47.5K, Resistor_SMD:R_0201_0603Metric_Pad0.64x0.40mm_HandSolder, symbol Device:R
- removed R5: 22.1K, Resistor_SMD:R_0201_0603Metric_Pad0.64x0.40mm_HandSolder, symbol Device:R
- removed R6, R7: 10K, Resistor_SMD:R_0201_0603Metric_Pad0.64x0.40mm_HandSolder, symbol Device:R
- removed R8: 31.6k, Resistor_SMD:R_0603_1608Metric, symbol Device:R
- removed R9: 10k, Resistor_SMD:R_0603_1608Metric, symbol Device:R
- removed U1: ESP32-WROOM-32, RF_Module:ESP32-WROOM-32, symbol RF_Module:ESP32-WROOM-32
- removed U2: CP2102N-Axx-xQFN28, Package_DFN_QFN:QFN-28-1EP_5x5mm_P0.5mm_EP3.35x3.35mm, symbol Interface_USB:CP2102N-Axx-xQFN28
- removed U4: USBLC6-2SC6, Package_TO_SOT_SMD:SOT-23-6, symbol Power_Protection:USBLC6-2SC6
- removed U5: MCP16301x-xCH, Package_TO_SOT_SMD:SOT-23-6, symbol Regulator_Switching:MCP16301x-xCH
- added U1, U2, U4, U5: PC817, Package_DIP:DIP-4_W7.62mm, symbol Isolator:PC817
- added U3: ESP32-DevKitC, PCM_Espressif:ESP32-DevKitC, symbol PCM_Espressif:ESP32-DevKitC
Connections:
- new net: U3.14 (GND), U3.32 (GND), U3.38 (GND)
Other:
- note removed: "5V-3.3V"
- note removed: "USB-Port"

Commit message: Relays
Parts:
- removed U1, U2, U4, U5: PC817, Package_DIP:DIP-4_W7.62mm, symbol Isolator:PC817
- added D10, D4, D6, D8: MRA4003T3G, Diode_SMD:D_SMA, symbol Diode:MRA4003T3G
- added D3, D5, D7, D9: LED, LED_SMD:LED_0603_1608Metric, symbol Device:LED
- added J2, J3, J4, J5: Screw_Terminal_01x03, TerminalBlock:TerminalBlock_MaiXu_MX126-5.0-03P_1x03_P5.00mm, symbol Connector:Screw_Terminal_01x03
- added J6: Screw_Terminal_01x02, TerminalBlock:TerminalBlock_MaiXu_MX126-5.0-02P_1x02_P5.00mm, symbol Connector:Screw_Terminal_01x02
- added K2, K3, K4, K5: SANYOU_SRD_Form_C, Relay_THT:Relay_SPDT_SANYOU_SRD_Series_Form_C, symbol Relay:SANYOU_SRD_Form_C
- added Q2, Q3, Q4, Q5: MMBT2222A, Package_TO_SOT_SMD:SOT-23, symbol Transistor_BJT:MMBT2222A
- added R10, R13, R4, R7: 1K, Resistor_SMD:R_0603_1608Metric, symbol Device:R
- added R11, R12, R14, R15, R5, R6, R8, R9: 10K, Resistor_SMD:R_0603_1608Metric, symbol Device:R
Connections:
- net +3V3: now reaches U3.1 (3V3)
- net GND: now reaches U3.14 (GND), U3.32 (GND), U3.38 (GND)
- net GND: now also J6.1 (Pin_1), Q2.2 (E), Q3.2 (E), Q4.2 (E), Q5.2 (E), R11.2, R14.2, R5.2, R8.2
- net +5V: now reaches U3.19 (5V)
- net +5V: now also D10.1 (K), D4.1 (K), D6.1 (K), D8.1 (K), J6.2 (Pin_2), K2.5, K3.5, K4.5, K5.5, R12.1, R15.1, R6.1, R9.1
- net SIG1: now reaches U3.30 (GPIO18)
- net SIG1: now also R7.1
- net SIG2: now reaches U3.31 (GPIO19)
- net SIG2: now also R4.1
- net SIG3: now reaches U3.33 (GPIO21)
- net SIG3: now also R10.1
- net SIG4: now reaches U3.36 (GPIO22)
- net SIG4: now also R13.1
- new net: D10.2 (A), D9.1 (K), K5.2, Q5.3 (C)
- new net: D5.1 (K), D6.2 (A), K3.2, Q3.3 (C)
- new net: Q4.1 (B), R10.2, R11.1
- new net: D7.1 (K), D8.2 (A), K4.2, Q4.3 (C)
- new net: J5.2 (Pin_2), K5.1
- new net: J5.1 (Pin_1), K5.3
- new net: J5.3 (Pin_3), K5.4
- new net: Q3.1 (B), R7.2, R8.1
- new net: Q2.1 (B), R4.2, R5.1
- new net: D9.2 (A), R15.2
- new net: D3.2 (A), R6.2
- new net: Q5.1 (B), R13.2, R14.1
- new net: J4.1 (Pin_1), K4.3
- new net: J4.2 (Pin_2), K4.1
- new net: J4.3 (Pin_3), K4.4
- new net: J2.2 (Pin_2), K2.1
- new net: D3.1 (K), D4.2 (A), K2.2, Q2.3 (C)
- new net: J2.1 (Pin_1), K2.3
- new net: J2.3 (Pin_3), K2.4
- new net: D7.2 (A), R12.2
- new net: D5.2 (A), R9.2
- new net: J3.1 (Pin_1), K3.3
- new net: J3.2 (Pin_2), K3.1
- new net: J3.3 (Pin_3), K3.4
Other:
- moved on the sheet: U3

Commit message: Schematic Redo
Parts:
- added J1: Input, TerminalBlock:TerminalBlock_MaiXu_MX126-5.0-05P_1x05_P5.00mm, symbol Connector:Screw_Terminal_01x05
- added R1, R16, R2, R3: 10k, Resistor_SMD:R_0603_1608Metric, symbol Device:R
Connections:
- net +3V3: now also R1.1, R16.1, R2.1, R3.1
- net GND: now also J1.5 (Pin_5)
- net SIG1: now also U3.29 (GPIO5); no longer U3.30 (GPIO18)
- net SIG2: now also U3.30 (GPIO18); no longer U3.31 (GPIO19)
- net SIG3: now also U3.31 (GPIO19); no longer U3.33 (GPIO21)
- net SIG4: now also U3.33 (GPIO21); no longer U3.36 (GPIO22)
- net IN3: now reaches U3.27 (GPIO16)
- net IN3: now also J1.2 (Pin_2), R2.2
- net IN4: now reaches U3.28 (GPIO17)
- net IN4: now also J1.1 (Pin_1), R1.2
- net IN2: now reaches U3.37 (GPIO23)
- net IN2: now also J1.3 (Pin_3), R3.2
- new net IN1: J1.4 (Pin_4), R16.2, U3.36 (GPIO22)
Other:
- title: ESP32 -> GateLink
- moved on the sheet: D10, D7, D8, D9, J4, J5, J6, K4, K5, Q4, Q5, R10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

Commit message: Change Pins for easier routing WIP PCB
Connections:
- net IN1: now also U3.37 (GPIO23); no longer U3.36 (GPIO22)
- net IN2: now also U3.36 (GPIO22); no longer U3.37 (GPIO23)
- net IN3: now also U3.28 (GPIO17); no longer U3.27 (GPIO16)
- net IN4: now also U3.27 (GPIO16); no longer U3.28 (GPIO17)
